File: KiCad/Amstrad-CPC-IO-Logger.kicad_pcb (KiCad board)
At the start: 2 copper layers, 89.1 x 74.4 mm, 20 parts, among them J1 Conn_02x25_Odd_Even, J2 Conn_02x02_Odd_Even, J3 Conn_02x04_Odd_Even, SW1 SW_Push, U1 Pico, U2 74LVC245, U3 74LVC245, U4 74LVC245, U5 74HCT00, U6 74HCT138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

Commit message: PCB Update to move the Pico to the edge of the PCB.
Parts:
- moved U1 8.39 mm to (115.8, 110.0)
- moved D1 8.28 mm to (97.0, 131.6)
Routing:
- net /~{IOWR}: track 61.0 -> 93.1 mm
- net /+5V: track 155.5 -> 176.8 mm
- net /GND: track 363.0 -> 344.1 mm
- net /~{ADHB_CE}: track 70.9 -> 52.7 mm
- net /P_D7: track 82.9 -> 65.7 mm
- net Net-(U8-E1): track 54.9 -> 40.2 mm
- net /P_A0: track 32.9 -> 45.2 mm
- net /A14: track 105.9 -> 116.9 mm
- net /P_A1: track 32.5 -> 43.2 mm
- net /A2: track 48.3 -> 39.5 mm
- net /A12: track 109.1 -> 100.2 mm
- net /P_A12: track 47.1 -> 38.3 mm, vias 1 -> 0
- net Net-(U1-RUN): track 36.7 -> 45.1 mm
- net /~{CSRD}: track 67.6 -> 59.2 mm, vias 1 -> 0
- net /P_D4: track 50.4 -> 42.1 mm
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Other:
- board text added: "RABS Amstrad CPC IO Logger V1.2"
- board text removed: "RABS Amstrad CPC IO Logger V1.1"
