File: KiCad/Amstrad-CPC-IO-Logger.kicad_pcb (KiCad board)
At the start: 2 copper layers, 89.1 x 74.4 mm, 20 parts, among them J1 Conn_02x25_Odd_Even, J2 Conn_02x02_Odd_Even, J3 Conn_02x04_Odd_Even, SW1 SW_Push, U1 Pico, U2 74LVC245, U3 74LVC245, U4 74LVC245, U5 74HCT00, U6 74HCT138, U7 74HCT32, U8 74HCT138

Commit message: Modifications for V2.0
Parts:
- added ?: , clipboard:ebb3ee9a-570f-4b0c-ad82-8a87958112c0, F.Cu at (105.3, 76.7)
- J3: value Conn_02x04_Odd_Even -> Conn_02x02_Odd_Even; footprint Connector_PinHeader_2.54mm:PinHeader_2x04_P2.54mm_Vertical -> Connector_PinHeader_2.54mm:PinHeader_2x02_P2.54mm_Vertical
- moved U1 0.13 mm to (115.8, 110.1)
- moved J3 0.13 mm to (134.5, 88.0)
Connections:
- U1 pad 24: /~{CTRL_CE} -> /~{P_DBGC}
- U1 pad 25: /~{ADHB_CE} -> /~{CTRL_CE}
- U1 pad 26: /~{DATA_CE} -> /~{ADHB_CE}
- U1 pad 27: /DATA_AB -> /~{DATA_CE}
- U1 pad 29: /~{P_CSRD} -> /DATA_AB
- U1 pad 31: /~{P_IOWR} -> /~{P_CSRD}
- U1 pad 32: unconnected-(U1-GPIO27_ADC1-Pad32)_1 -> /~{P_IOWR}
- U2 pad 14: unconnected-(U2-B4-Pad14) -> /~{P_DBGC}
- U2 pad 6: unconnected-(U2-A4-Pad6) -> /~{DBGC}
- U7 pad 3: Net-(U7-Pad3) -> /~{DBGC}
- U7 pad 4: Net-(U7-Pad3) -> /~{DBGC}
- U8 pad 12: /FB -> unconnected-(U8-O3-Pad12)
- U8 pad 13: /FA -> unconnected-(U8-O2-Pad13)
Routing:
- net /~{P_DBGC}: track 0.00 -> 64.4 mm, vias 0 -> 1
- net /~{CSRD}: track 59.2 -> 115.3 mm, vias 0 -> 1
- net /~{DBGC}: track 0.00 -> 54.4 mm
- net /~{IOWR}: track 93.1 -> 59.7 mm
- net /GND: track 344.1 -> 371.8 mm
- net /FB: track 26.1 -> 0.00 mm
- net /A13: track 103.2 -> 125.1 mm
- net /FA: track 21.5 -> 0.00 mm
- net /+5V: track 176.8 -> 158.1 mm
- net /A14: track 116.9 -> 133.8 mm
- net /A6: track 46.7 -> 61.0 mm, vias 1 -> 0
- net /~{CTRL_CE}: track 59.5 -> 46.7 mm
- net /P_A13: track 50.1 -> 62.3 mm, vias 1 -> 0
- net /P_A0: track 45.2 -> 34.5 mm
- net /A11: track 66.7 -> 56.2 mm
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Other:
- board size 89.1 x 74.4 mm -> 89.1 x 74.7 mm
- board text added: "RABS Amstrad CPC IO Logger V2.0"
- board text added: "https://github.com/rabs664/Amstrad-CPC-IO-Logger"
- board text removed: "FA"
- board text removed: "FB"
- board text removed: "RABS Amstrad CPC IO Logger V1.2"
