File: KiCad/Amstrad-CPC-IO-Logger.kicad_sch (KiCad schematic)
At the start: 20 parts, among them J1 Conn_02x25_Odd_Even, J2 Conn_02x02_Odd_Even, J3 Conn_02x04_Odd_Even, SW1 SW_Push, U1 Pico, U2 74LVC245, U3 74LVC245, U4 74LVC245, U5 74HCT00, U6 74HCT138, U7 74HCT32, U8 74HCT138

Commit message: Modifications for V2.0
Parts:
- removed J3: Conn_02x04_Odd_Even, Connector_PinHeader_2.54mm:PinHeader_2x04_P2.54mm_Vertical, symbol Connector_Generic:Conn_02x04_Odd_Even
- added J3: Conn_02x02_Odd_Even, Connector_PinHeader_2.54mm:PinHeader_2x02_P2.54mm_Vertical, symbol Connector_Generic:Conn_02x02_Odd_Even
Connections:
- net DATA_AB: now also U1.29 (GPIO22); no longer U1.27 (GPIO21)
- net F8: now also J3.1 (Pin_1)
- net F9: now also J3.3 (Pin_3)
- net ~{ADHB_CE}: now also U1.26 (GPIO20); no longer U1.25 (GPIO19)
- net ~{CSHB}: now also J3.2 (Pin_2), J3.4 (Pin_4)
- net ~{CTRL_CE}: now also U1.25 (GPIO19); no longer U1.24 (GPIO18)
- net ~{DATA_CE}: now also U1.27 (GPIO21); no longer U1.26 (GPIO20)
- net ~{P_CSRD}: now also U1.31 (GPIO26_ADC0); no longer U1.29 (GPIO22)
- net ~{P_IOWR}: now also U1.32 (GPIO27_ADC1); no longer U1.31 (GPIO26_ADC0)
- net ~{DBGC}: now reaches U7.3, U7.4
- net ~{DBGC}: now also U2.6 (A4)
- net ~{P_DBGC}: now reaches U2.14 (B4)
- net ~{P_DBGC}: now also U1.24 (GPIO18)
- net FA: no longer names the net of U8.13 (O2)
- net FB: no longer names the net of U8.12 (O3)
- no-connect marks 48 -> 47
Other:
- note added: "(~{CSRD}) provides a single Chip Select Read active low signal (i.e. combining IO Address, IORQ and RD)"
- note added: "(~{DBGC}) provides a signal for the explict 16-Bit IO Address associated with Debug Commands"
- note added: "(~{IORQ}) and (~{WR}) are combined to provide a single active low signal."
- note removed: "CSRD provides a single Chip Select Read active low signal (i.e. combining IO Address, IORQ and RD)"
- note removed: "IORQ and WR are combined to provide a single active low signal."
- moved on the sheet: U2
